File: GPS.kicad_sch (KiCad schematic)
At the start: 18 parts, among them J11 GPS_I2C, J2 RFPC-SMA28-F, SW4 GPS_RESET, U9 PA1616S_GPS

Commit message: done antenna
Parts:
- added C31: 1u, Capacitor_SMD:C_0603_1608Metric_Pad1.08x0.95mm_HandSolder, symbol Device:C
- added C32: 47p, Capacitor_SMD:C_0603_1608Metric_Pad1.08x0.95mm_HandSolder, symbol Device:C
- added L2: 33n, Inductor_SMD:L_0603_1608Metric_Pad1.05x0.95mm_HandSolder, symbol Device:L
- added R40: 10, Resistor_SMD:R_0603_1608Metric_Pad0.98x0.95mm_HandSolder, symbol Device:R
- J2: footprint RFPC-SMA28-F:GRADCONN_RFPC-SMA28-F -> TSOM Lib:GRADCONN_RFPC-SMA28-F
Connections:
- net +3V3: now also R40.1
- net GND: now also C31.2
- net GPS_EXT_OFF: now also C32.1; no longer J2.1
- new net: C31.1, L2.1, R40.2
- new net: C32.2, J2.1, L2.2
Other:
- moved on the sheet: J2

Commit message: did some stuff
Parts:
- C27, C28, C29: LCSC (none) -> C15849
- C30: LCSC (none) -> C14663
- C31: value 1u -> 10n; LCSC (none) -> C57112
- C32: LCSC (none) -> C1671
- D8: LCSC (none) -> C7371904
- L2: LCSC (none) -> C86068
- R24, R26: LCSC (none) -> C21190
- R25, R27, R28: LCSC (none) -> C25804
Changed lines of the file:
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@@
+			)
+		)
+		(property "LCSC" "C25804"
+			(at 212.09 100.584 0)
+			(effects
+				(font
+					(size 1.27 1.27)
+				)
+				(hide yes)
 			)
 		)
@@
 			)
 		)
-		(property "Value" "1u"
+		(property "Value" "10n"
 			(at 177.8 143.256 0)
 			(effects
@@
 		(property "P/N" "C0805C105J4RAC7210"
 			(at 173.99 142.24 0)
+			(effects
+				(font
+					(size 1.27 1.27)
+				)
+				(hide yes)
+			)
+		)
+		(property "LCSC" "C57112"
+			(at 176.784 140.97 0)
 			(effects
 				(font
@@
 			)
 		)
+		(property "LCSC" "C7371904"
+			(at 105.41 123.698 0)
+			(effects
+				(font
+					(size 1.27 1.27)
+				)
+				(hide yes)
+			)
+		)
 		(pin "2"
 		)
@@
 			)
 		)
+		(property "LCSC" "C15849"
+			(at 105.41 66.0399 0)
+			(effects
+				(font
+					(size 1.27 1.27)
+				)
+				(hide yes)
+			)
+		)
 		(pin "2"
 		)
@@
 			)
 		)
+		(property "LCSC" "C15849"
+			(at 94.234 107.95 0)
+			(effects
+				(font
+					(size 1.27 1.27)
+				)
+				(hide yes)
+			)
+		)
 		(pin "2"
 		)
@@
 		(property "P/N" "CRCW080510K0FKEA"
 			(at 115.57 83.82 0)
+			(effects
+				(font
+					(size 1.27 1.27)
+				)
+				(hide yes)
+			)
+		)
+		(property "LCSC" "C25804"
+			(at 112.395 82.677 0)
 			(effects
 				(font
@@
 			)
 		)
+		(property "LCSC" "C25804"
+			(at 202.438 97.282 0)
+			(effects
+				(font
+					(size 1.27 1.27)
+				)
+				(hide yes)
+			)
+		)
 		(pin "2"
 		)
@@
 			)
 		)
+		(property "LCSC" "C15849"
+			(at 99.314 92.71 0)
+			(effects
+				(font
+					(size 1.27 1.27)
+				)
+				(hide yes)
+			)
+		)
 		(pin "2"
 		)
@@
 			)
 		)
+		(property "LCSC" "C86068"
+			(at 182.88 133.35 0)
+			(effects
+				(font
+					(size 1.27 1.27)
+				)
+				(hide yes)
+			)
+		)
 		(pin "1"
 		)
@@
 			)
 		)
+		(property "LCSC" "C1671"
+			(at 208.534 127.7666 0)
+			(effects
+				(font
+					(size 1.27 1.27)
+				)
+				(hide yes)
+			)
+		)
 		(pin "2"
 		)
@@
 			)
 		)
+		(property "LCSC" "C21190"
+			(at 104.14 111.7599 0)
+			(effects
+				(font
+					(size 1.27 1.27)
+				)
+				(hide yes)
+			)
+		)
 		(pin "1"
 		)
@@
 			)
 		)
+		(property "LCSC" "C14663"
+			(at 115.57 66.0399 0)
+			(effects
+				(font
+					(size 1.27 1.27)
+				)
+				(hide yes)
+			)
+		)
 		(pin "2"
 		)
@@
 			(effects
 				(font
+					(size 1.27 1.27)
+				)
+				(hide yes)
+			)
+		)
+		(property "LCSC" "C21190"
+			(at 95.25 84.074 0)
+			(effects
+				(font

Commit message: gerb
Parts:
- FB1: footprint Resistor_SMD:R_0402_1005Metric -> Inductor_SMD:L_0603_1608Metric_Pad1.05x0.95mm_HandSolder
- R40: LCSC (none) -> C22859
Changed lines of the file:
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@@
 			)
 		)
-		(property "Footprint" "Resistor_SMD:R_0402_1005Metric"
+		(property "Footprint" "Inductor_SMD:L_0603_1608Metric_Pad1.05x0.95mm_HandSolder"
 			(at 99.822 55.88 90)
 			(effects
@@
 			(effects
 				(font
+					(size 1.27 1.27)
+				)
+				(hide yes)
+			)
+		)
+		(property "LCSC" "C22859"
+			(at 176.53 133.3499 0)
+			(effects
+				(font
