File: TSOMProject.kicad_sch (KiCad schematic)
At the start: 0 parts

Commit message: fix errors schem
Other:
- sheet FPGAConnector renamed Connector
- added sheet IMU (IMU.kicad_sch)
Changed lines of the file:
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@@
 			(color 0 0 0 0.0000)
 		)
-		(property "Sheetname" "FPGAConnector"
+		(property "Sheetname" "Connector"
 			(at 156.845 64.0584 0)
 			(effects
@@
 			(project "TSOMProject"
 				(path "/f13eb969-5de0-437e-a1b7-e0204111e0b2"
-					(page "1")
+					(page "2")
 				)
 			)
@@
 				)
 			)
+		)
+	)
+	(sheet
+		(at 163.195 32.385)
+		(size 47.625 23.495)
+		(exclude_from_sim no)
+		(in_bom yes)
+		(on_board yes)
+		(dnp no)
+		(fields_autoplaced yes)
+		(stroke
+			(width 0.1524)
+			(type solid)
+		)
+		(fill
+			(color 0 0 0 0.0000)
+		)
+		(property "Sheetname" "IMU"
+			(at 163.195 31.6734 0)
+			(effects
+				(font
+					(size 1.27 1.27)
+				)
+				(justify left bottom)
+			)
+		)
+		(property "Sheetfile" "IMU.kicad_sch"
+			(at 163.195 56.4646 0)
+			(effects
+				(font
+					(size 1.27 1.27)
+				)
+				(justify left top)
+			)
+		)
+		(instances
+			(project "TSOMProject"
+				(path "/f13eb969-5de0-437e-a1b7-e0204111e0b2"
+					(page "7")
+				)
+			)

Commit message: fin schematic
Other:
- added sheet Power Inputs (powerinputs.kicad_sch)
Changed lines of the file:
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@@
 	(paper "A4")
+	(sheet
+		(at 92.075 34.925)
+		(size 43.815 21.59)
+		(exclude_from_sim no)
+		(in_bom yes)
+		(on_board yes)
+		(dnp no)
+		(fields_autoplaced yes)
+		(stroke
+			(width 0.1524)
+			(type solid)
+		)
+		(fill
+			(color 0 0 0 0.0000)
+		)
+		(property "Sheetname" "Power Inputs"
+			(at 92.075 34.2134 0)
+			(effects
+				(font
+					(size 1.27 1.27)
+				)
+				(justify left bottom)
+			)
+		)
+		(property "Sheetfile" "powerinputs.kicad_sch"
+			(at 92.075 57.0996 0)
+			(effects
+				(font
+					(size 1.27 1.27)
+				)
+				(justify left top)
+			)
+		)
+		(instances
+			(project "TSOMProject"
+				(path "/f13eb969-5de0-437e-a1b7-e0204111e0b2"
+					(page "8")
+				)
+			)
+		)
+	)
 	(sheet
 		(at 156.845 64.77)

Commit message: im cooked
Other:
- removed sheet RF
Changed lines of the file:
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@@
-	)
-	(sheet
-		(at 158.115 106.68)
-		(size 57.785 33.655)
-		(exclude_from_sim no)
-		(in_bom yes)
-		(on_board yes)
-		(dnp no)
-		(fields_autoplaced yes)
-		(stroke
-			(width 0.1524)
-			(type solid)
-		)
-		(fill
-			(color 0 0 0 0.0000)
-		)
-		(property "Sheetname" "RF"
-			(at 158.115 105.9684 0)
-			(effects
-				(font
-					(size 1.27 1.27)
-				)
-				(justify left bottom)
-			)
-		)
-		(property "Sheetfile" "RF.kicad_sch"
-			(at 158.115 140.9196 0)
-			(effects
-				(font
-					(size 1.27 1.27)
-				)
-				(justify left top)
-			)
-		)
-		(instances
-			(project "TSOMProject"
-				(path "/f13eb969-5de0-437e-a1b7-e0204111e0b2"
-					(page "6")
-				)
-			)
-		)
 	)
 	(sheet
