File: untitled.kicad_sch (KiCad schematic)
At the start: 36 parts, among them U4 LT1963AEST-3.3#TRPBF, U5 TPS2115ADRBR, U6 TPS5405DR

Commit message: power/connectors
Parts:
- removed 3.3V1, 5V1: TestPoint, TestPoint:TestPoint_Pad_1.0x1.0mm, symbol Connector:TestPoint
- removed C10, C13, C20, C21, C22: 10uF, Capacitor_SMD:C_0805_2012Metric_Pad1.18x1.45mm_HandSolder, symbol Device:C
- removed C11, C12: 0.1uF, Capacitor_SMD:C_0603_1608Metric_Pad1.08x0.95mm_HandSolder, symbol Device:C
- removed C18: 1uF, Capacitor_SMD:C_0603_1608Metric_Pad1.08x0.95mm_HandSolder, symbol Device:C
- removed D3: MBR230S1F, Diode_SMD:D_SOD-123F, symbol Device:D_Schottky
- removed L1: 100uH, Inductor_SMD:L_Coilcraft_MSS1246-XXX, symbol Device:L
- removed R14: 332, Resistor_SMD:R_0603_1608Metric_Pad0.98x0.95mm_HandSolder, symbol Device:R
- removed R16: ROSC, Resistor_SMD:R_0603_1608Metric_Pad0.98x0.95mm_HandSolder, symbol Device:R
- removed R17: 10k, Resistor_SMD:R_0603_1608Metric_Pad0.98x0.95mm_HandSolder, symbol Device:R
- removed U4: LT1963AEST-3.3#TRPBF, Package_TO_SOT_SMD:SOT-223-3_TabPin2, symbol Regulator_Linear:LT1963AxST-3.3
- removed U5: TPS2115ADRBR, TPS2115ABDR:SON65P300X300X100-9N, symbol TPS2115ADBR:TPS2115ADRBR
- removed U6: TPS5405DR, UTSVT_Power:TPS5405DR, symbol UTSVT-Power:TPS5405DR
- added D12: SS14, Diode_SMD:D_SMA, symbol Diode:SS14
- added L2: 33uH, symbol Device:L
- added R42, R43, R44: 100k, symbol Device:R
- added U4: LMR16006YQ5, Package_TO_SOT_SMD:SOT-23-6, symbol Regulator_Switching:LMR16006YQ5
- C14: value 10uF -> 47uF; footprint Capacitor_SMD:C_0805_2012Metric_Pad1.18x1.45mm_HandSolder -> (none); Mouser Part Number GRM21BR61H106KE43K -> (none); P/N GRM21BR61H106KE43K -> (none)
- C15: value 1uF -> 10uF; footprint Capacitor_SMD:C_0603_1608Metric_Pad1.08x0.95mm_HandSolder -> (none); Mouser Part Number MLASU168SB5105KTNA01 -> (none); P/N MLASU168SB5105KTNA01 -> (none)
- C16: value 10nF -> 10uF; footprint Capacitor_SMD:C_0603_1608Metric_Pad1.08x0.95mm_HandSolder -> (none); Mouser Part Number MSASH168SB5103KTNA01 -> (none); P/N MSASH168SB5103KTNA01 -> (none)
- C17: value 3.3nF -> 100nF; footprint Capacitor_SMD:C_0603_1608Metric_Pad1.08x0.95mm_HandSolder -> (none); Mouser Part Number 06035C332K4T2A -> (none); P/N 06035C332K4T2A -> (none)
- C19: value 0.1uF -> 10uF; footprint Capacitor_SMD:C_0603_1608Metric_Pad1.08x0.95mm_HandSolder -> (none); Mouser Part Number MLASH168SB7104KTNA01 -> (none); P/N MLASH168SB7104KTNA01 -> (none)
- R15: value 16k -> 100k; footprint Resistor_SMD:R_0603_1608Metric_Pad0.98x0.95mm_HandSolder -> (none); Mouser Part Number CRCW060316K0FKEA -> (none); P/N CRCW060316K0FKTA -> (none)
Connections:
- net +24V: now also R15.1; no longer C15.1
- net +3V3: no longer C14.1
- net GND: now also C16.1, R43.2, R44.2, U4.2 (GND); no longer R15.2
- net +12V: now reaches C19.1
- net +12V: now also D12.1 (K)
- net at C17.1: now also U4.1 (CB)
- net at C19.2: now also R42.2, R43.1, R44.1, U4.3 (FB)
- net at C17.2: now also L2.1, R42.1, U4.6 (SW); no longer R15.1
- new net: C14.1, R15.2, U4.5 (VIN)
- new net: C15.1, U4.4 (~{SHDN})
- new net: D12.2 (A), L2.2
- no-connect marks 1 -> 0
Other:
- note removed: "5->3.3v LDO"
- note removed: "5v Power Mux"
- note removed: "Cout > 33.8uF -> 30uF For 30uF, ESR < 120mΩ"
- note removed: "DNP for 120 kHz switching frequency"
- note removed: "ILim(A) = 500/R 1.5A = 500/332"
- note removed: "Max current: 1.5A"
- note removed: "Prioritizes IN1 (Buck)"

Commit message: fix errors schem
Parts:
- removed C14: 47uF, symbol Device:C
- removed C15, C16, C19: 10uF, symbol Device:C
- removed C17: 100nF, symbol Device:C
- removed D12: SS14, Diode_SMD:D_SMA, symbol Diode:SS14
- removed D19: USB, LED_SMD:LED_0603_1608Metric_Pad1.05x0.95mm_HandSolder, symbol Device:LED
- removed D20: BUCK, LED_SMD:LED_0603_1608Metric_Pad1.05x0.95mm_HandSolder, symbol Device:LED
- removed D4: 24V, LED_SMD:LED_0603_1608Metric_Pad1.05x0.95mm_HandSolder, symbol Device:LED
- removed R15, R42, R43, R44: 100k, symbol Device:R
- removed R18: 4.3k, Resistor_SMD:R_0603_1608Metric_Pad0.98x0.95mm_HandSolder, symbol Device:R
- removed R28, R34: 768, Resistor_SMD:R_0603_1608Metric_Pad0.98x0.95mm_HandSolder, symbol Device:R
- removed U4: LMR16006YQ5, Package_TO_SOT_SMD:SOT-23-6, symbol Regulator_Switching:LMR16006YQ5
- added C40: 10uF, symbol Device:C
- added C44: 47uF, symbol Device:C_Polarized_US
- added C_BOOT1: 100nF, symbol Device:C
- added C_COMP1: 560pF, symbol Device:C
- added C_COMP2: 6.8pF, symbol Device:C
- added D12: 550mV, Package_TO_SOT_SMD:SOT-363_SC-70-6, symbol Diode:SD103ATW
- added R_COMP1: 44.2k, symbol Device:R_US
- added R_FBB1: 10.5k, symbol Device:R_US
- added R_FBT1: 147k, symbol Device:R_US
- added R_t1: 105k, symbol Device:R_US
- added U10: TPS54560BDDA, Package_SO:Texas_R-PDSO-G8_EP2.95x4.9mm_Mask2.4x3.1mm_ThermalVias, symbol Regulator_Switching:TPS54560BDDA
- L2: value 33uH -> 8.2uH
Connections:
- net +24V is gone; now on net +12V: R20.1
- net +5V is gone; now on net +12V: R21.1
- net FAULT is gone; now on net +12V: D6.1 (K)
- net GND is gone; now on net +12V: D5.1 (K)
- net STAT is gone; now on net +12V: D7.1 (K)
- net +12V: now also L2.2, C40.1, C40.2, C44.1, C44.2, C_COMP1.2, C_COMP2.2, D12.6 (A), R_FBB1.2, R_FBT1.1, R_t1.2, U10.2 (VIN), U10.7 (GND), U10.9 (GND)
- net at L2.1: now also C_BOOT1.2, D12.1 (K), U10.8 (SW)
- new net: R_FBB1.1, R_FBT1.2, U10.5 (FB)
- new net: C_BOOT1.1, U10.1 (BOOT)
- new net: R_t1.1, U10.4 (RT/CLK)
- new net: C_COMP2.1, R_COMP1.1, U10.6 (COMP)
- new net: C_COMP1.1, R_COMP1.2
- no-connect marks 0 -> 1
Other:
- removed sheet Power Protection
- note added: ". The EN pin has an internal pullup current source, I1, of 1.2 μA that enables operation of the TPS54560B when the EN pin floats."
- note added: "24->12v Buck Converter"
- note removed: "24->5v Buck Converter"

Commit message: only da inductor
Parts:
- C40, C44, C_BOOT1, C_COMP1, C_COMP2, R_COMP1, R_FBB1, R_FBT1, R_t1: footprint (none) -> Capacitor_SMD:C_0603_1608Metric_Pad1.08x0.95mm_HandSolder
- R19, R20, R21: footprint Resistor_SMD:R_0603_1608Metric_Pad0.98x0.95mm_HandSolder -> Capacitor_SMD:C_0603_1608Metric_Pad1.08x0.95mm_HandSolder
Changed lines of the file:
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@@
 			)
 		)
-		(property "Footprint" ""
+		(property "Footprint" "Capacitor_SMD:C_0603_1608Metric_Pad1.08x0.95mm_HandSolder"
 			(at 134.366 71.374 90)
 			(effects
@@
 			)
 		)
-		(property "Footprint" ""
+		(property "Footprint" "Capacitor_SMD:C_0603_1608Metric_Pad1.08x0.95mm_HandSolder"
 			(at 134.366 54.864 90)
 			(effects
@@
 			)
 		)
-		(property "Footprint" ""
+		(property "Footprint" "Capacitor_SMD:C_0603_1608Metric_Pad1.08x0.95mm_HandSolder"
 			(at 54.356 59.944 90)
 			(effects
@@
 			)
 		)
-		(property "Footprint" ""
+		(property "Footprint" "Capacitor_SMD:C_0603_1608Metric_Pad1.08x0.95mm_HandSolder"
 			(at 151.13 64.77 0)
 			(effects
@@
 			)
 		)
-		(property "Footprint" "Resistor_SMD:R_0603_1608Metric_Pad0.98x0.95mm_HandSolder"
+		(property "Footprint" "Capacitor_SMD:C_0603_1608Metric_Pad1.08x0.95mm_HandSolder"
 			(at 221.742 34.925 90)
 			(effects
@@
 			)
 		)
-		(property "Footprint" ""
+		(property "Footprint" "Capacitor_SMD:C_0603_1608Metric_Pad1.08x0.95mm_HandSolder"
 			(at 40.3352 63.5 0)
 			(effects
@@
 			)
 		)
-		(property "Footprint" ""
+		(property "Footprint" "Capacitor_SMD:C_0603_1608Metric_Pad1.08x0.95mm_HandSolder"
 			(at 112.7252 50.8 0)
 			(effects
@@
 			)
 		)
-		(property "Footprint" ""
+		(property "Footprint" "Capacitor_SMD:C_0603_1608Metric_Pad1.08x0.95mm_HandSolder"
 			(at 54.3052 73.66 0)
 			(effects
@@
 			)
 		)
-		(property "Footprint" "Resistor_SMD:R_0603_1608Metric_Pad0.98x0.95mm_HandSolder"
+		(property "Footprint" "Capacitor_SMD:C_0603_1608Metric_Pad1.08x0.95mm_HandSolder"
 			(at 201.422 34.925 90)
 			(effects
@@
 			)
 		)
-		(property "Footprint" "Resistor_SMD:R_0603_1608Metric_Pad0.98x0.95mm_HandSolder"
+		(property "Footprint" "Capacitor_SMD:C_0603_1608Metric_Pad1.08x0.95mm_HandSolder"
 			(at 211.582 34.925 90)
 			(effects
@@
 			)
 		)
-		(property "Footprint" ""
+		(property "Footprint" "Capacitor_SMD:C_0603_1608Metric_Pad1.08x0.95mm_HandSolder"
 			(at 65.7352 69.85 0)
 			(effects
@@
 			)
 		)
-		(property "Footprint" ""
+		(property "Footprint" "Capacitor_SMD:C_0603_1608Metric_Pad1.08x0.95mm_HandSolder"
 			(at 75.946 68.834 90)
 			(effects

Commit message: im cooked
Connections:
- net +12V: no longer C40.1, C40.2, C44.2, C_COMP1.2, C_COMP2.2, D12.6 (A), D5.1 (K), D6.1 (K), D7.1 (K), R20.1, R_FBB1.2, R_t1.2, U10.2 (VIN), U10.7 (GND), U10.9 (GND)
- new net +24V: C40.1, R20.1, U10.2 (VIN)
- new net GND: C40.2, C44.2, C_COMP1.2, C_COMP2.2, D12.6 (A), D5.1 (K), D6.1 (K), D7.1 (K), R_FBB1.2, R_t1.2, U10.7 (GND), U10.9 (GND)
Changed lines of the file:
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@@
-	)
-	(junction
-		(at 171.45 50.8)
-		(diameter 0)
-		(color 0 0 0 0)
 	)
 	(junction
@@
 	)
 	(junction
-		(at 151.13 76.2)
-		(diameter 0)
-		(color 0 0 0 0)
-	)
-	(junction
 		(at 88.9 76.2)
 		(diameter 0)
@@
 	)
 	(junction
-		(at 30.48 45.72)
-		(diameter 0)
-		(color 0 0 0 0)
-	)
-	(junction
 		(at 133.35 76.2)
 		(diameter 0)
@@
 	(junction
 		(at 151.13 50.8)
-		(diameter 0)
-		(color 0 0 0 0)
-	)
-	(junction
-		(at 39.37 76.2)
 		(diameter 0)
 		(color 0 0 0 0)
@@
 	(wire
 		(pts
-			(xy 30.48 76.2) (xy 39.37 76.2)
-		)
-		(stroke
-			(width 0)
-			(type default)
-		)
-	)
-	(wire
-		(pts
 			(xy 203.2 48.895) (xy 203.2 51.435)
 		)
@@
 	(wire
 		(pts
-			(xy 171.45 76.2) (xy 151.13 76.2)
-		)
-		(stroke
-			(width 0)
-			(type default)
-		)
-	)
-	(wire
-		(pts
-			(xy 30.48 45.72) (xy 30.48 76.2)
-		)
-		(stroke
-			(width 0)
-			(type default)
-		)
-	)
-	(wire
-		(pts
 			(xy 53.34 53.34) (xy 53.34 55.88)
 		)
@@
 		)
 		(stroke
-			(width 0)
-			(type default)
-		)
-	)
-	(wire
-		(pts
-			(xy 171.45 50.8) (xy 171.45 76.2)
-		)
-		(stroke
