File: CAN.kicad_sch (KiCad schematic)
At the start: 18 parts, among them IC1 TCAN337DCNR, IC2 TCAN337DCNR, U7 CDSOT23-T24CAN, U8 CDSOT23-T24CAN

Commit message: fix errors schem
Parts:
- renumbered R11 to R10
Connections:
- net CARCAN_Fault: no longer names the net of R11.1
- no-connect marks 2 -> 3
Other:
- moved on the sheet: CC_FLT1, CC_Term1, R11, R12, R22

Commit message: only da inductor
Parts:
- R10, R11, R12, R13, R22, R23: footprint Resistor_SMD:R_0603_1608Metric_Pad0.98x0.95mm_HandSolder -> Capacitor_SMD:C_0603_1608Metric_Pad1.08x0.95mm_HandSolder
Changed lines of the file:
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@@
 			)
 		)
-		(property "Footprint" "Resistor_SMD:R_0603_1608Metric_Pad0.98x0.95mm_HandSolder"
+		(property "Footprint" "Capacitor_SMD:C_0603_1608Metric_Pad1.08x0.95mm_HandSolder"
 			(at 26.162 35.56 90)
 			(effects
@@
 			)
 		)
-		(property "Footprint" "Resistor_SMD:R_0603_1608Metric_Pad0.98x0.95mm_HandSolder"
+		(property "Footprint" "Capacitor_SMD:C_0603_1608Metric_Pad1.08x0.95mm_HandSolder"
 			(at 205.74 132.842 90)
 			(effects
@@
 			)
 		)
-		(property "Footprint" "Resistor_SMD:R_0603_1608Metric_Pad0.98x0.95mm_HandSolder"
+		(property "Footprint" "Capacitor_SMD:C_0603_1608Metric_Pad1.08x0.95mm_HandSolder"
 			(at 148.082 91.44 90)
 			(effects
@@
 			)
 		)
-		(property "Footprint" "Resistor_SMD:R_0603_1608Metric_Pad0.98x0.95mm_HandSolder"
+		(property "Footprint" "Capacitor_SMD:C_0603_1608Metric_Pad1.08x0.95mm_HandSolder"
 			(at 237.617 88.265 90)
 			(effects
@@
 			)
 		)
-		(property "Footprint" "Resistor_SMD:R_0603_1608Metric_Pad0.98x0.95mm_HandSolder"
+		(property "Footprint" "Capacitor_SMD:C_0603_1608Metric_Pad1.08x0.95mm_HandSolder"
 			(at 83.82 75.692 90)
 			(effects
@@
 			)
 		)
-		(property "Footprint" "Resistor_SMD:R_0603_1608Metric_Pad0.98x0.95mm_HandSolder"
+		(property "Footprint" "Capacitor_SMD:C_0603_1608Metric_Pad1.08x0.95mm_HandSolder"
 			(at 115.062 41.91 90)
 			(effects

Commit message: start layout
Other:
- note added: "Car CAN Bus Termination"
Changed lines of the file:
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@@
 		)
 	)
-	(text "Telemetry CAN Bus Termination"
+	(text "Car CAN Bus Termination"
 		(exclude_from_sim no)
 		(at 89.154 72.644 0)

Commit message: more layout
Connections:
- net CarCAN_Fault: now also R11.1
- net CarCAN_H renamed CarCAN_H+
- net CarCAN_L renamed CarCAN_L-
- net TelCAN_H renamed TelCAN_H+
- net TelCAN_L renamed TelCAN_L-
- no-connect marks 3 -> 2
Changed lines of the file:
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@@
 	)
 	(junction
-		(at 206.375 90.17)
+		(at 205.74 90.17)
 		(diameter 0)
 		(color 0 0 0 0)
@@
 	)
 	(no_connect
-		(at 116.84 35.56)
-	)
-	(no_connect
 		(at 165.735 97.79)
 	)
@@
 	(wire
 		(pts
-			(xy 206.375 103.505) (xy 208.915 103.505)
+			(xy 205.74 103.505) (xy 208.915 103.505)
 		)
 		(stroke
@@
 	(wire
 		(pts
-			(xy 206.375 90.17) (xy 206.375 103.505)
+			(xy 205.74 90.17) (xy 205.74 103.505)
 		)
 		(stroke
@@
 	(wire
 		(pts
-			(xy 206.375 90.17) (xy 212.09 90.17)
+			(xy 205.74 90.17) (xy 212.09 90.17)
 		)
 		(stroke
@@
 	(wire
 		(pts
-			(xy 191.135 90.17) (xy 206.375 90.17)
+			(xy 191.135 90.17) (xy 205.74 90.17)
 		)
 		(stroke
@@
 		)
 	)
+	(label "CarCAN_Fault"
+		(at 116.84 35.56 0)
+		(effects
+			(font
+				(size 1.27 1.27)
+			)
+			(justify left bottom)
+		)
+	)
 	(label "TelCAN_Fault"
 		(at 239.395 81.28 0)
@@
 		)
 	)
-	(global_label "TelCAN_L"
+	(global_label "TelCAN_L-"
 		(shape input)
 		(at 212.09 95.25 0)
@@
 		)
 		(property "Intersheetrefs" "${INTERSHEET_REFS}"
-			(at 223.4814 95.25 0)
+			(at 225.0538 95.25 0)
 			(effects
 				(font
@@
 		)
 	)
-	(global_label "CarCAN_L"
+	(global_label "CarCAN_L-"
 		(shape input)
 		(at 101.6 77.47 0)
@@
 		)
 		(property "Intersheetrefs" "${INTERSHEET_REFS}"
-			(at 113.4752 77.47 0)
+			(at 115.0476 77.47 0)
 			(effects
 				(font
@@
 		)
 	)
-	(global_label "CarCAN_H"
+	(global_label "CarCAN_H+"
 		(shape input)
 		(at 78.74 77.47 180)
@@
 		)
 		(property "Intersheetrefs" "${INTERSHEET_REFS}"
-			(at 66.5624 77.47 0)
+			(at 64.99 77.47 0)
 			(effects
 				(font
@@
 		)
 	)
-	(global_label "TelCAN_H"
+	(global_label "TelCAN_H+"
 		(shape input)
 		(at 212.09 90.17 0)
@@
 		)
 		(property "Intersheetrefs" "${INTERSHEET_REFS}"
-			(at 223.7838 90.17 0)
+			(at 225.3562 90.17 0)
 			(effects
 				(font
@@
 		)
 	)
-	(global_label "CarCAN_L"
+	(global_label "CarCAN_L-"
 		(shape input)
 		(at 90.17 39.37 0)
@@
 		)
 		(property "Intersheetrefs" "${INTERSHEET_REFS}"
-			(at 102.0452 39.37 0)
+			(at 103.6176 39.37 0)
 			(effects
 				(font
@@
 		)
 	)
-	(global_label "CarCAN_H"
+	(global_label "CarCAN_H+"
 		(shape input)
 		(at 90.17 34.29 0)
@@
 		)
 		(property "Intersheetrefs" "${INTERSHEET_REFS}"
-			(at 102.3476 34.29 0)
+			(at 103.92 34.29 0)
 			(effects
 				(font
@@
 		)
 	)
-	(global_label "TelCAN_H"
+	(global_label "TelCAN_H+"
 		(shape input)
 		(at 200.66 134.62 180)
@@
 		)
 		(property "Intersheetrefs" "${INTERSHEET_REFS}"
-			(at 188.9662 134.62 0)
+			(at 187.3938 134.62 0)
 			(effects
 				(font
@@
 		)
 	)
-	(global_label "TelCAN_L"
+	(global_label "TelCAN_L-"
 		(shape input)
 		(at 222.25 134.62 0)
@@
 		)
 		(property "Intersheetrefs" "${INTERSHEET_REFS}"
-			(at 233.6414 134.62 0)
-			(effects
-				(font
+			(at 235.2138 134.62 0)
+			(effects
+				(font
