File: FPGAConnector.kicad_sch (KiCad schematic)
At the start: 1 part

Commit message: power/connectors
Parts:
- removed FPGA_Connector1: ~, symbol FPGA_Connector:FPGA_Connector
- added CPU_Connector, FPGA_Connector: ~, symbol FPGA_Connector:FPGA_Connector
Changed lines of the file:
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@@
 	(paper "A4")
 	(symbol
+		(lib_name "FPGA_Connector_1")
 		(lib_id "FPGA_Connector:FPGA_Connector")
-		(at 146.05 93.98 0)
+		(at 124.46 55.88 0)
 		(unit 1)
 		(exclude_from_sim no)
@@
 		(on_board yes)
 		(dnp no)
-		(fields_autoplaced yes)
-		(property "Reference" "FPGA_Connector1"
-			(at 147.32 80.01 0)
+		(property "Reference" "CPU_Connector"
+			(at 131.572 41.656 0)
 			(effects
 				(font
 					(size 1.27 1.27)
 				)
-				(justify left)
 			)
 		)
 		(property "Value" "~"
-			(at 160.02 95.2499 0)
+			(at 124.46 40.64 0)
 			(effects
 				(font
 					(size 1.27 1.27)
 				)
-				(justify left)
 			)
 		)
 		(property "Footprint" ""
-			(at 146.05 93.98 0)
+			(at 124.46 55.88 0)
 			(effects
 				(font
@@
 		)
 		(property "Datasheet" ""
-			(at 146.05 93.98 0)
+			(at 124.46 55.88 0)
 			(effects
 				(font
@@
 		)
 		(property "Description" ""
-			(at 146.05 93.98 0)
+			(at 124.46 55.88 0)
 			(effects
 				(font
@@
 			)
 		)
-		(pin "7"
+		(pin "3"
 		)
 		(pin "1"
@@
 		(pin "4"
 		)
-		(pin "3"
+		(pin "8"
 		)
 		(pin "5"
 		)
-		(pin "8"
+		(pin "11"
 		)
 		(pin "6"
 		)
+		(pin "7"
+		)
+		(pin "12"
+		)
+		(pin "9"
+		)
+		(pin "10"
+		)
 		(instances
-			(project ""
+			(project "TSOMProject"
 				(path "/f13eb969-5de0-437e-a1b7-e0204111e0b2/555dcf2f-9cf7-4916-9b4f-3a8f620095c0"
-					(reference "FPGA_Connector1")
+					(reference "CPU_Connector")
 					(unit 1)
 				)
-				(path "/f13eb969-5de0-437e-a1b7-e0204111e0b2/5da8fdf4-ad8c-47df-b08e-df168b9b0cb6"
-					(reference "FPGA_Connector1")
+			)
+		)
+	)
+	(symbol
+		(lib_name "FPGA_Connector_2")
+		(lib_id "FPGA_Connector:FPGA_Connector")
+		(at 119.38 95.25 0)
+		(unit 1)
+		(exclude_from_sim no)
+		(in_bom yes)
+		(on_board yes)
+		(dnp no)
+		(property "Reference" "FPGA_Connector"
+			(at 126.492 81.026 0)
+			(effects
+				(font
+					(size 1.27 1.27)
+				)
+			)
+		)
+		(property "Value" "~"
+			(at 119.38 80.01 0)
+			(effects
+				(font
+					(size 1.27 1.27)
+				)
+			)
+		)
+		(property "Footprint" ""
+			(at 119.38 95.25 0)
+			(effects
+				(font
+					(size 1.27 1.27)
+				)
+				(hide yes)
+			)
+		)
+		(property "Datasheet" ""
+			(at 119.38 95.25 0)
+			(effects
+				(font
+					(size 1.27 1.27)
+				)
+				(hide yes)
+			)
+		)
+		(property "Description" ""
+			(at 119.38 95.25 0)
+			(effects
+				(font
+					(size 1.27 1.27)
+				)
+				(hide yes)
+			)
+		)
+		(pin "3"
+		)
+		(pin "1"
+		)
+		(pin "2"
+		)
+		(pin "4"
+		)
+		(pin "8"
+		)
+		(pin "5"
+		)
+		(pin "11"
+		)
+		(pin "6"
+		)
+		(pin "7"
+		)
+		(pin "12"
+		)
+		(pin "9"
+		)
+		(pin "10"
+		)
+		(instances
+			(project "TSOMProject"
+				(path "/f13eb969-5de0-437e-a1b7-e0204111e0b2/555dcf2f-9cf7-4916-9b4f-3a8f620095c0"
+					(reference "FPGA_Connector")
 					(unit 1)
 				)

Commit message: fix errors schem
Parts:
- removed CPU_Connector, FPGA_Connector: ~, symbol FPGA_Connector:FPGA_Connector
- added J4: Conn_02x06_Counter_Clockwise, symbol Connector_Generic:Conn_02x06_Counter_Clockwise
- added J5: MX150_02x10_Vertical, UTSVT_Connectors:MX150_02x10_Vertical, symbol utsvt_connectors:MX150_02x10_Vertical
- added J6: To The Zedboard, symbol Connector_Generic:Conn_02x06_Counter_Clockwise
- added J7: Debug, symbol Connector_Generic:Conn_02x06_Counter_Clockwise
- added J8: Conn_02x06_Odd_Even, symbol Connector_Generic:Conn_02x06_Odd_Even
Connections:
- new net +24V: J5.1 (Fusebox+), J5.14 (+24V), J5.4 (+24V)
- new net +3V3: J4.6 (Pin_6), J4.7 (Pin_7), J6.6 (Pin_6), J6.7 (Pin_7), J7.6 (Pin_6), J7.7 (Pin_7), J8.1 (Pin_1), J8.2 (Pin_2)
- new net CarCAN_H: J5.2 (CANH_IN)
- new net CarCAN_RX: J5.3 (CANL_IN), J8.11 (Pin_11)
- new net CarCAN_TX: J5.12 (CANH_OUT), J5.13 (CANL_OUT), J8.5 (Pin_5)
- new net GND: J4.5 (Pin_5), J4.8 (Pin_8), J5.11 (Fusebox-), J5.17 (GND), J5.7 (GND), J6.5 (Pin_5), J6.8 (Pin_8), J7.5 (Pin_5), J7.8 (Pin_8), J8.3 (Pin_3), J8.4 (Pin_4)
- new net GPS_SCL: J4.3 (Pin_3)
- new net GPS_SDA: J4.4 (Pin_4)
- new net IMU_CLK: J4.9 (Pin_9)
- new net IMU_CS: J4.12 (Pin_12)
- new net IMU_MISO: J4.10 (Pin_10)
- new net IMU_MOSI: J4.1 (Pin_1)
- new net RF_RX: J4.11 (Pin_11)
- new net RF_TX: J4.2 (Pin_2)
- new net T10: J6.10 (Pin_10), J7.10 (Pin_10)
- new net TP1: J6.1 (Pin_1), J7.1 (Pin_1)
- new net TP11: J6.11 (Pin_11), J7.11 (Pin_11)
- new net TP12: J6.12 (Pin_12), J7.12 (Pin_12)
- new net TP2: J6.2 (Pin_2), J7.2 (Pin_2)
- new net TP3: J6.3 (Pin_3), J7.3 (Pin_3)
- new net TP4: J6.4 (Pin_4), J7.4 (Pin_4)
- new net TP9: J6.9 (Pin_9), J7.9 (Pin_9)
- new net TelCAN_RX: J5.5 (TELH_IN), J5.6 (TELL_IN), J8.9 (Pin_9)
- new net TelCAN_TX: J5.15 (TELH_OUT), J5.16 (TELL_OUT), J8.7 (Pin_7)
- no-connect marks 0 -> 10
Other:
- note added: "CPU Connector"
- note added: "FPGA Connector"
- note added: "FPGA Test Points"
- note added: "For reference to MIO PMOD on the Zedboard, pin 11 corresponds to JE1 pin 9 corresponds to JE2 pin 7 corresponds to JE3 pin 5 corresponds to JE4 pin 3 corresponds to GND pin 1 corresponds to 3V3 pin 12 corresponds to JE7 pin 10 corresponds to JE6 pin 8 corresponds to JE9 pin 6 corresponds to JE10 pin 4 corresponds to JE11 pin 2 corresponds to JE12"
- note added: "MX150 Connector"

Commit message: only da inductor
Parts:
- removed J7: Debug, symbol Connector_Generic:Conn_02x06_Counter_Clockwise
- added J9: Conn_02x05_Counter_Clockwise, Connector_PinHeader_2.54mm:PinHeader_2x05_P2.54mm_Vertical, symbol Connector_Generic:Conn_02x05_Counter_Clockwise
- J4: footprint (none) -> Connector_PinHeader_2.54mm:PinHeader_2x07_P2.54mm_Vertical
- J5: value MX150_02x10_Vertical -> Conn_02x07_Vertical; footprint UTSVT_Connectors:MX150_02x10_Vertical -> UTSVT_Connectors:Molex_Microfit3.0_02x07_14-Pin-Vertical-PCB-Receptacle_447691401; symbol utsvt_connectors:MX150_02x10_Vertical -> Connector_Generic:Conn_02x07_Top_Bottom
- J6, J8: footprint (none) -> Connector_PinHeader_2.54mm:PinHeader_2x06_P2.54mm_Vertical
Connections:
- net TP11 is gone; now on net TP4: J6.11 (Pin_11)
- net +24V: now also J5.11 (Pin_11), J5.8 (Pin_8); no longer J5.14 (+24V)
- net +3V3: now also J9.5 (Pin_5), J9.6 (Pin_6)
- net CarCAN_TX: now also J5.10 (Pin_10), J5.9 (Pin_9); no longer J5.12 (CANH_OUT), J5.13 (CANL_OUT)
- net GND: now also J5.14 (Pin_14), J9.4 (Pin_4), J9.7 (Pin_7); no longer J5.11 (Fusebox-), J5.17 (GND)
- net TP1: now also J6.2 (Pin_2), J9.1 (Pin_1); no longer J6.1 (Pin_1)
- net TP2: now also J6.3 (Pin_3), J9.2 (Pin_2); no longer J6.2 (Pin_2)
- net TP3: now also J6.4 (Pin_4), J9.3 (Pin_3); no longer J6.3 (Pin_3)
- net TP4: now also J9.10 (Pin_10); no longer J6.4 (Pin_4)
- net TelCAN_TX: now also J5.12 (Pin_12), J5.13 (Pin_13); no longer J5.15 (TELH_OUT), J5.16 (TELL_OUT)
- net T10 renamed TP5
- net TP5: now also J9.9 (Pin_9)
- net TP12 renamed IMU_INT2
- net TP9 renamed TP6
- net TP6: now also J9.8 (Pin_8)
- new net IMU_INT1: J6.1 (Pin_1)
- no-connect marks 10 -> 4

Commit message: im cooked
Connections:
- net RF_RX is gone; now on net +3V3: J4.11 (Pin_11)
- net RF_TX is gone; now on net IMU_CS: J4.2 (Pin_2)
- net +3V3: now also J4.12 (Pin_12), J6.11 (Pin_11), J6.12 (Pin_12); no longer J4.6 (Pin_6), J4.7 (Pin_7), J6.6 (Pin_6), J6.7 (Pin_7)
- net GND: now also J4.10 (Pin_10), J4.9 (Pin_9), J6.10 (Pin_10), J6.9 (Pin_9); no longer J4.5 (Pin_5), J4.8 (Pin_8), J6.5 (Pin_5), J6.8 (Pin_8)
- net GPS_SCL: now also J4.5 (Pin_5); no longer J4.3 (Pin_3)
- net GPS_SDA: now also J4.7 (Pin_7); no longer J4.4 (Pin_4)
- net IMU_CLK: now also J4.8 (Pin_8); no longer J4.9 (Pin_9)
- net IMU_CS: no longer J4.12 (Pin_12)
- net IMU_INT2: now also J6.2 (Pin_2); no longer J6.12 (Pin_12)
- net IMU_MISO: now also J4.6 (Pin_6); no longer J4.10 (Pin_10)
- net TP1: now also J6.3 (Pin_2); no longer J6.2 (Pin_2)
- net TP2: now also J6.5 (Pin_5); no longer J6.3 (Pin_3)
- net TP3: now also J6.7 (Pin_7); no longer J6.4 (Pin_4)
- net TP4: now also J6.4 (Pin_4); no longer J6.11 (Pin_11)
- net TP5: now also J6.6 (Pin_6); no longer J6.10 (Pin_10)
- net TP6: now also J6.8 (Pin_8); no longer J6.9 (Pin_9)
- no-connect marks 4 -> 6
Changed lines of the file:
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@@
+	)
+	(no_connect
+		(at 199.39 63.5)
 	)
 	(no_connect
@@
 	)
 	(no_connect
+		(at 186.69 63.5)
+	)
+	(no_connect
 		(at 133.35 132.08)
 	)
@@
 	(wire
 		(pts
-			(xy 177.8 63.5) (xy 186.69 63.5)
-		)
-		(stroke
-			(width 0)
-			(type default)
-		)
-	)
-	(wire
-		(pts
 			(xy 201.93 118.11) (xy 212.09 118.11)
 		)
@@
 		(pts
 			(xy 245.11 115.57) (xy 252.73 115.57)
-		)
-		(stroke
-			(width 0)
-			(type default)
-		)
-	)
-	(wire
-		(pts
-			(xy 199.39 63.5) (xy 207.01 63.5)
 		)
 		(stroke
@@
 		)
 	)
-	(label "RF_UART_RX"
-		(at 201.93 63.5 0)
-		(effects
-			(font
-				(size 0.762 0.762)
-			)
-			(justify left bottom)
-		)
-	)
 	(label "TP6"
 		(at 252.73 115.57 0)
@@
 	(label "TP6"
 		(at 209.55 115.57 0)
-		(effects
-			(font
-				(size 0.762 0.762)
-			)
-			(justify left bottom)
-		)
-	)
-	(label "RF_UART_TX"
-		(at 177.8 63.5 0)
 		(effects
 			(font
@@
 		)
 	)
-	(global_label "RF_RX"
-		(shape input)
-		(at 207.01 63.5 0)
-		(fields_autoplaced yes)
-		(effects
-			(font
-				(size 1.27 1.27)
-			)
-			(justify left)
-		)
-		(property "Intersheetrefs" "${INTERSHEET_REFS}"
-			(at 215.8009 63.5 0)
-			(effects
-				(font
-					(size 1.27 1.27)
-				)
-				(justify left)
-				(hide yes)
-			)
-		)
-	)
 	(global_label "GPS_SDA"
 		(shape input)
@@
 		(property "Intersheetrefs" "${INTERSHEET_REFS}"
 			(at 102.5458 129.54 0)
-			(effects
-				(font
-					(size 1.27 1.27)
-				)
-				(justify right)
-				(hide yes)
-			)
-		)
-	)
-	(global_label "RF_TX"
-		(shape input)
-		(at 177.8 63.5 180)
-		(fields_autoplaced yes)
-		(effects
-			(font
-				(size 1.27 1.27)
-			)
-			(justify right)
-		)
-		(property "Intersheetrefs" "${INTERSHEET_REFS}"
-			(at 169.3115 63.5 0)
 			(effects
 				(font
@@
 	)
 	(symbol
-		(lib_id "power:GND")
-		(at 181.61 118.11 0)
-		(unit 1)
-		(exclude_from_sim no)
-		(in_bom yes)
-		(on_board yes)
-		(dnp no)
-		(fields_autoplaced yes)
-		(property "Reference" "#PWR017"
-			(at 181.61 124.46 0)
-			(effects
-				(font
-					(size 1.27 1.27)
-				)
-				(hide yes)
-			)
-		)
-		(property "Value" "GND"
-			(at 181.61 123.19 0)
-			(effects
-				(font
-					(size 1.27 1.27)
-				)
-				(hide yes)
-			)
-		)
-		(property "Footprint" ""
-			(at 181.61 118.11 0)
-			(effects
-				(font
-					(size 1.27 1.27)
-				)
-				(hide yes)
-			)
-		)
-		(property "Datasheet" ""
-			(at 181.61 118.11 0)
-			(effects
-				(font
-					(size 1.27 1.27)
-				)
-				(hide yes)
-			)
-		)
-		(property "Description" "Power symbol creates a global label with name \"GND\" , ground"
-			(at 181.61 118.11 0)
-			(effects
-				(font
-					(size 1.27 1.27)
-				)
-				(hide yes)
-			)
-		)
-		(pin "1"
-		)
-		(instances
-			(project "TSOMProject"
-				(path "/f13eb969-5de0-437e-a1b7-e0204111e0b2/555dcf2f-9cf7-4916-9b4f-3a8f620095c0"
-					(reference "#PWR017")
-					(unit 1)
-				)
-			)
-		)
-	)
-	(symbol
 		(lib_id "power:+24V")
 		(at 208.28 73.66 180)
@@
 			)
 		)
-		(property "Datasheet" "~"
+		(property "Datasheet" "https://files.digilent.com/resources/programmable-logic/zedboard/ZedBoard_HW_UG_v2_2.pdf"
 			(at 194.31 113.03 0)
 			(effects
@@
 					(unit 1)
 				)
+			)
+		)
+	)
+	(symbol
+		(lib_id "power:GND")
+		(at 181.61 118.11 0)
+		(unit 1)
+		(exclude_from_sim no)
+		(in_bom yes)
+		(on_board yes)
+		(dnp no)
+		(fields_autoplaced yes)
+		(property "Reference" "#PWR017"
+			(at 181.61 124.46 0)
+			(effects
+				(font
+					(size 1.27 1.27)
+				)
+				(hide yes)
+			)
+		)
+		(property "Value" "GND"
+			(at 181.61 123.19 0)
+			(effects
+				(font
+					(size 1.27 1.27)
+				)
+			)
+		)
+		(property "Footprint" ""
+			(at 181.61 118.11 0)
+			(effects
+				(font
+					(size 1.27 1.27)
+				)
+				(hide yes)
+			)
+		)
+		(property "Datasheet" ""
+			(at 181.61 118.11 0)
+			(effects
+				(font
+					(size 1.27 1.27)
+				)
+				(hide yes)
+			)
+		)
+		(property "Description" "Power symbol creates a global label with name \"GND\" , ground"
+			(at 181.61 118.11 0)
+			(effects
+				(font
+					(size 1.27 1.27)
+				)
+				(hide yes)
+			)
+		)
+		(pin "1"
+		)
+		(instances
+			(project ""
+				(path "/f13eb969-5de0-437e-a1b7-e0204111e0b2/555dcf2f-9cf7-4916-9b4f-3a8f620095c0"
+					(reference "#PWR017")
+					(unit 1)
+				)

Commit message: more layout
Parts:
- J4: footprint Connector_PinHeader_2.54mm:PinHeader_2x07_P2.54mm_Vertical -> Connector_PinHeader_2.54mm:PinHeader_2x06_P2.54mm_Vertical
Connections:
- net CarCAN_RX: now also J8.7 (Pin_7); no longer J5.3 (Pin_3), J8.11 (Pin_11)
- net CarCAN_TX: now also J8.9 (Pin_9); no longer J5.10 (Pin_10), J5.9 (Pin_9), J8.5 (Pin_5)
- net GPS_SCL: now also J4.7 (Pin_7); no longer J4.5 (Pin_5)
- net GPS_SDA: now also J4.5 (Pin_5); no longer J4.7 (Pin_7)
- net IMU_CLK: now also J6.1 (Pin_1); no longer J4.8 (Pin_8)
- net IMU_CS: now also J6.3 (Pin_2); no longer J4.2 (Pin_2)
- net IMU_INT1: now also J6.6 (Pin_6); no longer J6.1 (Pin_1)
- net IMU_INT2: now also J6.5 (Pin_5); no longer J6.2 (Pin_2)
- net IMU_MISO: now also J6.4 (Pin_4); no longer J4.6 (Pin_6)
- net IMU_MOSI: now also J6.2 (Pin_2); no longer J4.1 (Pin_1)
- net TP1: now also J4.1 (Pin_1); no longer J6.3 (Pin_2)
- net TP2: now also J4.6 (Pin_6), J9.10 (Pin_10); no longer J6.5 (Pin_5), J9.2 (Pin_2)
- net TP3: no longer J6.7 (Pin_7)
- net TP4: now also J4.2 (Pin_2), J9.2 (Pin_2); no longer J6.4 (Pin_4), J9.10 (Pin_10)
- net TP5: now also J4.8 (Pin_8); no longer J6.6 (Pin_6)
- net TP6: no longer J6.8 (Pin_8)
- net TelCAN_RX: now also J8.5 (Pin_5); no longer J5.5 (Pin_5), J5.6 (Pin_6), J8.9 (Pin_9)
- net TelCAN_TX: now also J8.11 (Pin_11); no longer J5.12 (Pin_12), J5.13 (Pin_13), J8.7 (Pin_7)
- net CarCAN_H renamed CarCAN_H+
- net CarCAN_H+: now also J5.9 (Pin_9)
- new net CarCAN_L-: J5.10 (Pin_10), J5.3 (Pin_3)
- new net TelCAN_H+: J5.12 (Pin_12), J5.5 (Pin_5)
- new net TelCAN_L-: J5.13 (Pin_13), J5.6 (Pin_6)
- no-connect marks 6 -> 8
Other:
- note added: "For reference to MIO PMOD on the Zedboard, pin 11 corresponds to JE1 pin 9 corresponds to JE2 pin 7 corresponds to JE3 pin 5 corresponds to JE4 pin 3 corresponds to GND pin 1 corresponds to 3V3 pin 12 corresponds to JE7 pin 10 corresponds to JE8 pin 8 corresponds to JE9 pin 6 corresponds to JE10 pin 4 corresponds to JE11 pin 2 corresponds to JE12"
- note removed: "For reference to MIO PMOD on the Zedboard, pin 11 corresponds to JE1 pin 9 corresponds to JE2 pin 7 corresponds to JE3 pin 5 corresponds to JE4 pin 3 corresponds to GND pin 1 corresponds to 3V3 pin 12 corresponds to JE7 pin 10 corresponds to JE6 pin 8 corresponds to JE9 pin 6 corresponds to JE10 pin 4 corresponds to JE11 pin 2 corresponds to JE12"
