File: IMU.kicad_sch (KiCad schematic)
At the start: 4 parts, among them U1 ASM330LHHTR

Commit message: only da inductor
Parts:
- U1: footprint ASM330LHHTR-IMU:LGA-14L_2P5X3X0P83_STM -> KiCad:LSM6DS3USTR
Connections:
- net IMU_INT1: now reaches U1.4 (INT1)
- net IMU_INT2: now reaches U1.9 (INT2)
- no-connect marks 2 -> 0
Changed lines of the file:
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@@
 		(color 0 0 0 0)
 	)
-	(no_connect
-		(at 146.05 86.36)
-	)
-	(no_connect
-		(at 100.33 81.28)
-	)
 	(wire
 		(pts
@@
 	(wire
 		(pts
-			(xy 97.79 78.74) (xy 99.06 78.74)
+			(xy 85.09 78.74) (xy 99.06 78.74)
 		)
 		(stroke
@@
 			)
 			(justify right bottom)
+		)
+	)
+	(global_label "IMU_INT1"
+		(shape input)
+		(at 100.33 81.28 180)
+		(effects
+			(font
+				(size 1.27 1.27)
+			)
+			(justify right)
+		)
+		(property "Intersheetrefs" "${INTERSHEET_REFS}"
+			(at 100.33 81.28 0)
+			(effects
+				(font
+					(size 1.27 1.27)
+				)
+				(hide yes)
+			)
 		)
 	)
@@
 				)
 				(justify left)
+				(hide yes)
+			)
+		)
+	)
+	(global_label "IMU_INT2"
+		(shape input)
+		(at 146.05 86.36 0)
+		(effects
+			(font
+				(size 1.27 1.27)
+			)
+			(justify left)
+		)
+		(property "Intersheetrefs" "${INTERSHEET_REFS}"
+			(at 146.05 86.36 0)
+			(effects
+				(font
+					(size 1.27 1.27)
+				)
 				(hide yes)
 			)
@@
 			)
 		)
-		(property "Footprint" "ASM330LHHTR-IMU:LGA-14L_2P5X3X0P83_STM"
+		(property "Footprint" "KiCad:LSM6DS3USTR"
 			(at 100.33 73.66 0)
 			(effects
@@
 	(symbol
 		(lib_id "power:GND")
-		(at 97.79 78.74 0)
+		(at 85.09 78.74 0)
 		(unit 1)
 		(exclude_from_sim no)
@@
 		(dnp no)
 		(property "Reference" "#PWR04"
-			(at 97.79 85.09 0)
+			(at 85.09 85.09 0)
 			(effects
 				(font
@@
 		)
 		(property "Value" "GND"
-			(at 93.98 79.248 0)
+			(at 81.28 79.248 0)
 			(effects
 				(font
@@
 		)
 		(property "Footprint" ""
-			(at 97.79 78.74 0)
+			(at 85.09 78.74 0)
 			(effects
 				(font
@@
 		)
 		(property "Datasheet" ""
-			(at 97.79 78.74 0)
+			(at 85.09 78.74 0)
 			(effects
 				(font
@@
 		)
 		(property "Description" "Power symbol creates a global label with name \"GND\" , ground"
-			(at 97.79 78.74 0)
-			(effects
-				(font
+			(at 85.09 78.74 0)
+			(effects
+				(font

Commit message: more layout
Connections:
- net +3.3V: no longer C4.1
- net GND: no longer C4.2
Other:
- moved on the sheet: C3, C4
Changed lines of the file:
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@@
 	(symbol
 		(lib_id "Device:C")
-		(at 161.29 95.25 0)
+		(at 130.81 102.87 0)
 		(unit 1)
 		(exclude_from_sim no)
@@
 		(fields_autoplaced yes)
 		(property "Reference" "C4"
-			(at 165.1 93.9799 0)
+			(at 134.62 101.5999 0)
 			(effects
 				(font
@@
 		)
 		(property "Value" "100nf"
-			(at 165.1 96.5199 0)
+			(at 134.62 104.1399 0)
 			(effects
 				(font
@@
 		)
 		(property "Footprint" "Capacitor_SMD:C_0603_1608Metric_Pad1.08x0.95mm_HandSolder"
-			(at 162.2552 99.06 0)
+			(at 131.7752 106.68 0)
 			(effects
 				(font
@@
 		)
 		(property "Datasheet" "~"
-			(at 161.29 95.25 0)
+			(at 130.81 102.87 0)
 			(effects
 				(font
@@
 		)
 		(property "Description" "Unpolarized capacitor 100nf"
-			(at 161.29 95.25 0)
+			(at 130.81 102.87 0)
 			(effects
 				(font
@@
 		)
 		(property "Sim.Device" ""
-			(at 161.29 95.25 0)
+			(at 130.81 102.87 0)
 			(effects
 				(font
@@
 		)
 		(property "Sim.Library" ""
-			(at 161.29 95.25 0)
+			(at 130.81 102.87 0)
 			(effects
 				(font
@@
 		)
 		(property "Sim.Name" ""
-			(at 161.29 95.25 0)
+			(at 130.81 102.87 0)
 			(effects
 				(font
@@
 		)
 		(property "P/N" "MLASH168SB7104KTNA01"
-			(at 161.29 95.25 0)
+			(at 130.81 102.87 0)
 			(effects
 				(font
@@
 	(symbol
 		(lib_id "Device:C")
-		(at 149.86 95.25 0)
+		(at 161.29 95.25 0)
 		(unit 1)
 		(exclude_from_sim no)
@@
 		(fields_autoplaced yes)
 		(property "Reference" "C3"
-			(at 153.67 93.9799 0)
+			(at 165.1 93.9799 0)
 			(effects
 				(font
@@
 		)
 		(property "Value" "10uf"
-			(at 153.67 96.5199 0)
+			(at 165.1 96.5199 0)
 			(effects
 				(font
@@
 		)
 		(property "Footprint" "Capacitor_SMD:C_0603_1608Metric_Pad1.08x0.95mm_HandSolder"
-			(at 150.8252 99.06 0)
+			(at 162.2552 99.06 0)
 			(effects
 				(font
@@
 		)
 		(property "Datasheet" "~"
-			(at 149.86 95.25 0)
+			(at 161.29 95.25 0)
 			(effects
 				(font
@@
 		)
 		(property "Description" "Unpolarized capacitor 10uf"
-			(at 149.86 95.25 0)
+			(at 161.29 95.25 0)
 			(effects
 				(font
@@
 		)
 		(property "P/N" "GRM21BR61H106KE43K"
-			(at 149.86 95.25 0)
+			(at 161.29 95.25 0)
 			(effects
 				(font
@@
 		)
 		(property "Sim.Device" ""
-			(at 149.86 95.25 0)
+			(at 161.29 95.25 0)
 			(effects
 				(font
@@
 		)
 		(property "Sim.Library" ""
-			(at 149.86 95.25 0)
+			(at 161.29 95.25 0)
 			(effects
 				(font
@@
 		)
 		(property "Sim.Name" ""
-			(at 149.86 95.25 0)
-			(effects
-				(font
+			(at 161.29 95.25 0)
+			(effects
+				(font
