File: IMU.kicad_sch (KiCad schematic)
At the start: 4 parts, among them U1 ASM330LHHTR

Commit message: did some stuff
Parts:
- C1, C4: LCSC (none) -> C14663
- C3: LCSC (none) -> C440198
- U1: LCSC (none) -> C459826
Changed lines of the file:
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@@
+			)
+		)
+		(property "LCSC" "C14663"
+			(at 153.67 93.9799 0)
+			(effects
+				(font
+					(size 1.27 1.27)
+				)
+				(hide yes)
 			)
 		)
@@
 			)
 		)
+		(property "LCSC" "C459826"
+			(at 123.19 63.5 0)
+			(effects
+				(font
+					(size 1.27 1.27)
+				)
+				(hide yes)
+			)
+		)
 		(pin "1"
 		)
@@
 			)
 		)
+		(property "LCSC" "C440198"
+			(at 165.1 93.9799 0)
+			(effects
+				(font
+					(size 1.27 1.27)
+				)
+				(hide yes)
+			)
+		)
 		(pin "1"
 		)
@@
 			(effects
 				(font
+					(size 1.27 1.27)
+				)
+				(hide yes)
+			)
+		)
+		(property "LCSC" "C14663"
+			(at 85.09 93.218 0)
+			(effects
+				(font
