File: TSOMProject.kicad_pcb (KiCad board)
At the start: 2 copper layers, 60 parts, among them J1 RF_UART, J11 GPS_I2C, Q1 NMOS, SW1 RF_RESET, SW2 RF_COM, SW4 GPS_RESET, U10 TPS54560BDDA

Commit message: only da inductor
Parts:
- added BAT1: ML414, DataAcqGPS:BAT_2994TR, F.Cu at (126.8, 42.0)
- added IC1: TCAN337DCNR, UTSVT_ICs:TCAN337DCNR, F.Cu at (140.8, 72.5)
- added IC2: TCAN337DCNR, UTSVT_ICs:TCAN337DCNR, F.Cu at (140.8, 77.0)
- added J10: Conn_02x02_Odd_Even, Connector_Molex:Molex_Nano-Fit_105310-xx04_2x02_P2.50mm_Vertical, F.Cu at (88.0, 36.5)
- added J12: GPS_BAT, UTSVT_Special:TestPoint_HEX_3mmID, F.Cu at (108.0, 106.0)
- added J5: Conn_02x07_Vertical, UTSVT_Connectors:Molex_Microfit3.0_02x07_14-Pin-Vertical-PCB-Receptacle_447691401, F.Cu at (163.5, 43.0)
- added J8: Conn_02x06_Odd_Even, Connector_PinHeader_2.54mm:PinHeader_2x06_P2.54mm_Vertical, F.Cu at (213.6, 84.9)
- added U1: ASM330LHHTR, KiCad:LSM6DS3USTR, F.Cu at (198.8, 41.2)
- added U7: CDSOT23-T24CAN, UTSVT_ICs:CDSOT23-T24CAN, F.Cu at (135.7, 72.7)
- added U8: CDSOT23-T24CAN, UTSVT_ICs:CDSOT23-T24CAN, F.Cu at (135.7, 77.4)
- added U9: PA1616S_GPS, DataAcqGPS:PA1616S_ADA, F.Cu at (112.7, 31.3)
- added X1: DigiXBeeRX900Micro, RF_Module:Digi_XBee_SMT, F.Cu at (65.5, 55.4)
- moved SW1 12.9 mm to (100.1, 49.0), turned to 180 degrees

Commit message: start layout
Parts:
- added C40: 10uF, Capacitor_SMD:C_0603_1608Metric_Pad1.08x0.95mm_HandSolder, B.Cu at (187.0, 142.2)
- added C44: 47uF, Capacitor_SMD:C_0603_1608Metric_Pad1.08x0.95mm_HandSolder, B.Cu at (162.5, 146.0)
- added C6: 470 uF, Capacitor_SMD:C_0603_1608Metric_Pad1.08x0.95mm_HandSolder, F.Cu at (133.7, 92.0)
- added C_BOOT1: 100nF, Capacitor_SMD:C_0603_1608Metric_Pad1.08x0.95mm_HandSolder, B.Cu at (182.0, 137.6)
- added C_COMP1: 560pF, Capacitor_SMD:C_0603_1608Metric_Pad1.08x0.95mm_HandSolder, B.Cu at (185.5, 153.2)
- added C_COMP2: 6.8pF, Capacitor_SMD:C_0603_1608Metric_Pad1.08x0.95mm_HandSolder, B.Cu at (172.0, 144.0)
- added F1: +4A, Fuse:Fuseholder_Blade_Mini_Keystone_3568, F.Cu at (169.8, 94.8)
- added F2: +5A, Fuse:Fuseholder_Blade_Mini_Keystone_3568, F.Cu at (147.8, 91.7)
- added J14: Barrel_Jack_Switch, KiCad:694108301002, F.Cu at (147.8, 99.3)
- added J2: Conn_Coaxial, Connector_Coaxial:U.FL_Molex_MCRF_73412-0110_Vertical, F.Cu at (145.7, 158.0)
- added J3: Conn_Coaxial, Connector_Coaxial:U.FL_Molex_MCRF_73412-0110_Vertical, F.Cu at (182.4, 128.4)
- added J4: Conn_02x06_Counter_Clockwise, Connector_PinHeader_2.54mm:PinHeader_2x07_P2.54mm_Vertical, F.Cu at (204.5, 112.2)
- added J6: To The Zedboard, Connector_PinHeader_2.54mm:PinHeader_2x06_P2.54mm_Vertical, F.Cu at (204.2, 133.6)
- added J9: Conn_02x05_Counter_Clockwise, Connector_PinHeader_2.54mm:PinHeader_2x05_P2.54mm_Vertical, F.Cu at (197.2, 134.6)
- added R_COMP1: 44.2k, Capacitor_SMD:C_0603_1608Metric_Pad1.08x0.95mm_HandSolder, B.Cu at (185.0, 148.7)
- added R_FBB1: 10.5k, Capacitor_SMD:C_0603_1608Metric_Pad1.08x0.95mm_HandSolder, B.Cu at (167.0, 146.0)
- added R_FBT1: 147k, Capacitor_SMD:C_0603_1608Metric_Pad1.08x0.95mm_HandSolder, B.Cu at (169.0, 145.7)
- added R_t1: 105k, Capacitor_SMD:C_0603_1608Metric_Pad1.08x0.95mm_HandSolder, B.Cu at (183.0, 144.5)
- C27, C28, C29, C30, C31, C32, C33, C34, C35: footprint Capacitor_SMD:C_0805_2012Metric -> Capacitor_SMD:C_0603_1608Metric_Pad1.08x0.95mm_HandSolder
- D12, D5, D6, D7, J10, U10: moved to B.Cu
- R10, R11, R12, R13, R22, R23: footprint Resistor_SMD:R_0603_1608Metric_Pad0.98x0.95mm_HandSolder -> Capacitor_SMD:C_0603_1608Metric_Pad1.08x0.95mm_HandSolder
- R19, R20, R21: footprint Resistor_SMD:R_0603_1608Metric_Pad0.98x0.95mm_HandSolder -> Capacitor_SMD:C_0603_1608Metric_Pad1.08x0.95mm_HandSolder; moved to B.Cu
- R24, R25, R26, R29, R30, R31, R32, R33, R35, R36, R37, R38, R39, R40, R41: footprint Resistor_SMD:R_0805_2012Metric -> Capacitor_SMD:C_0603_1608Metric_Pad1.08x0.95mm_HandSolder
- moved C4 121.5 mm to (207.6, 158.0), turned to -90 degrees
- moved C3 120.7 mm to (205.0, 158.0), turned to -90 degrees
- moved C1 118.3 mm to (199.1, 159.4), turned to -90 degrees
- moved J5 115.6 mm to (159.7, 158.6)
- moved D5 114.4 mm to (193.0, 138.7), turned to 90 degrees
- moved U1 113.8 mm to (199.5, 155.1)
- moved X1 110.8 mm to (138.3, 139.0), turned to -90 degrees
- moved D6 110.1 mm to (189.5, 138.7), turned to 90 degrees
- moved R19 108.6 mm to (193.0, 134.3), turned to -90 degrees
- moved D7 105.7 mm to (186.0, 138.5), turned to 90 degrees
- moved U9 104.9 mm to (169.2, 119.7), turned to -90 degrees
- moved R20 104.3 mm to (189.5, 134.3), turned to -90 degrees
- moved J10 103.4 mm to (175.3, 91.8), turned to -90 degrees
- moved C23 103.2 mm to (189.7, 130.1), turned to -90 degrees
- moved C24 102.5 mm to (191.2, 130.1), turned to -90 degrees
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
Commit message: im cooked
Parts:
- removed C31: 10u, Capacitor_SMD:C_0603_1608Metric_Pad1.08x0.95mm_HandSolder
- removed C32, C34, C35: 1u, Capacitor_SMD:C_0603_1608Metric_Pad1.08x0.95mm_HandSolder
- removed C33: 47p, Capacitor_SMD:C_0603_1608Metric_Pad1.08x0.95mm_HandSolder
- removed D10: RF_ON, LED_SMD:LED_0805_2012Metric
- removed D11: RF_COM_LED, LED_SMD:LED_0805_2012Metric
- removed D9: RF_RSSI, LED_SMD:LED_0805_2012Metric
- removed J1: RF_UART, Connector_PinHeader_2.54mm:PinHeader_1x03_P2.54mm_Vertical
- removed J2: Conn_Coaxial, Connector_Coaxial:U.FL_Molex_MCRF_73412-0110_Vertical
- removed Q1: NMOS, Package_TO_SOT_SMD:SOT-23-3
- removed R29, R31, R32, R35, R37, R38, R41: 10k, Capacitor_SMD:C_0603_1608Metric_Pad1.08x0.95mm_HandSolder
- removed R30, R33, R36, R39, R40: 1k, Capacitor_SMD:C_0603_1608Metric_Pad1.08x0.95mm_HandSolder
- removed SW1: RF_RESET, Button_Switch_SMD:SW_SPST_B3SL-1002P
- removed SW2: RF_COM, Button_Switch_SMD:SW_SPST_B3SL-1002P
- removed X1: DigiXBeeRX900Micro, RF_Module:Digi_XBee_SMT
- moved C_COMP1 74.8 mm to (143.6, 91.3), turned to 90 degrees
- moved R_COMP1 66.9 mm to (144.1, 95.8), turned to 90 degrees
- moved D5 65.8 mm to (136.1, 105.8), turned to -90 degrees
- moved CC_Term2 62.9 mm to (164.9, 148.2), turned to 180 degrees
- moved R19 61.8 mm to (136.1, 110.2), turned to 90 degrees
- moved C40 60.1 mm to (142.1, 102.3), turned to 90 degrees
- moved D6 59.8 mm to (139.6, 105.8), turned to -90 degrees
- moved R12 59.8 mm to (167.4, 148.2), turned to 90 degrees
- moved R_t1 57.8 mm to (146.1, 100.0), turned to -90 degrees
- moved R20 55.5 mm to (139.6, 110.2), turned to 90 degrees
- moved U7 54.8 mm to (170.4, 146.4), turned to 180 degrees
- moved D7 53.8 mm to (143.1, 106.0), turned to -90 degrees
- moved U10 49.6 mm to (151.7, 101.0), turned to 0 degrees
- moved R21 49.1 mm to (143.1, 110.3), turned to 90 degrees
- moved IC2 49.0 mm to (175.1, 145.9)
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Connections:
- BAT1 pad N: +12V -> GND
- C1 pad 2: +12V -> GND
- C23 pad 2: +12V -> GND
- C24 pad 2: +12V -> GND
- C25 pad 2: +12V -> GND
- C26 pad 2: +12V -> GND
- C27 pad 2: +12V -> GND
- C28 pad 2: +12V -> GND
- C29 pad 2: +12V -> GND
- C3 pad 2: +12V -> GND
- C30 pad 2: +12V -> GND
- C4 pad 2: +12V -> GND
- C40 pad 1: +12V -> +24V
- C40 pad 2: +12V -> GND
- C44 pad 2: +12V -> GND
- C6 pad 2: +12V -> GND
- CC_FLT1 pad 1: +12V -> GND
- CC_FLT2 pad 1: +12V -> GND
- C_COMP1 pad 2: +12V -> GND
- C_COMP2 pad 2: +12V -> GND
- D12 pad 6: +12V -> GND
- D5 pad 1: +12V -> GND
- D6 pad 1: +12V -> GND
- D7 pad 1: +12V -> GND
- D8 pad 1: +12V -> GND
- IC1 pad 2: +12V -> GND
- IC2 pad 2: +12V -> GND
- J10 pad 2: +12V -> GND
- J14 pad 2: +12V -> GND
- J3 pad 2: +12V -> GND
- J4 pad 10: IMU_MISO -> GND
- J4 pad 11: RF_RX -> +3V3
- J4 pad 12: IMU_CS -> +3V3
- J4 pad 2: RF_TX -> IMU_CS
- J4 pad 3: GPS_SCL -> unconnected-(J4-Pin_3-Pad3)
- J4 pad 4: GPS_SDA -> unconnected-(J4-Pin_4-Pad4)
- J4 pad 5: +12V -> GPS_SCL
- J4 pad 6: +3V3 -> IMU_MISO
- J4 pad 7: +3V3 -> GPS_SDA
- J4 pad 8: +12V -> IMU_CLK
- J4 pad 9: IMU_CLK -> GND
- J5 pad 1: +12V -> +24V
- J5 pad 11: +12V -> +24V
- J5 pad 14: +12V -> GND
- J5 pad 4: +12V -> +24V
- J5 pad 7: +12V -> GND
- J5 pad 8: +12V -> +24V
- J6 pad 10: /Connector/TP5 -> GND
- J6 pad 11: /Connector/TP4 -> +3V3
- J6 pad 12: IMU_INT2 -> +3V3
- J6 pad 2: /Connector/TP1 -> IMU_INT2
- J6 pad 3: /Connector/TP2 -> /Connector/TP1
- J6 pad 4: /Connector/TP3 -> /Connector/TP4
- J6 pad 5: +12V -> /Connector/TP2
- J6 pad 6: +3V3 -> /Connector/TP5
- J6 pad 7: +3V3 -> /Connector/TP3
- J6 pad 8: +12V -> /Connector/TP6
- J6 pad 9: /Connector/TP6 -> GND
- J8 pad 3: +12V -> GND
- J8 pad 4: +12V -> GND
- J9 pad 4: +12V -> GND
- J9 pad 7: +12V -> GND
- R20 pad 1: +12V -> +24V
- R_FBB1 pad 2: +12V -> GND
- R_t1 pad 2: +12V -> GND
- SW4 pad 1: +12V -> GND
- U1 pad 2: +12V -> GND
- U1 pad 3: +12V -> GND
- U1 pad 6: +12V -> GND
- U1 pad 7: +12V -> GND
- U10 pad 2: +12V -> +24V
- U10 pad 7: +12V -> GND
- U10 pad 9: +12V -> GND
- U7 pad 3: +12V -> GND
- U8 pad 3: +12V -> GND
- U9 pad 12: +12V -> GND
- U9 pad 19: +12V -> GND
- U9 pad 3: +12V -> GND
- U9 pad 8: +12V -> GND

Commit message: more layout
Parts:
- added H1: M.3, MountingHole:MountingHole_3mm, F.Cu at (138.4, 89.4)
- added H2: M.3, MountingHole:MountingHole_3mm, F.Cu at (138.4, 157.8)
- added H3: M.3, MountingHole:MountingHole_3mm, F.Cu at (205.4, 89.6)
- added H4: M.3, MountingHole:MountingHole_3mm, F.Cu at (205.4, 157.6)
- C23, C24, CC_FLT1, CC_Term2, IC2, R10, R11, R12, U7: moved to B.Cu
- J4: footprint Connector_PinHeader_2.54mm:PinHeader_2x07_P2.54mm_Vertical -> Connector_PinHeader_2.54mm:PinHeader_2x06_P2.54mm_Vertical
- moved C25 50.1 mm to (187.9, 96.6)
- moved CC_Term2 49.1 mm to (188.6, 105.1)
- moved C26 47.0 mm to (187.9, 98.2)
- moved R13 45.7 mm to (183.6, 94.2)
- moved R23 45.7 mm to (183.5, 92.6)
- moved CC_FLT2 44.8 mm to (183.5, 91.0), turned to 0 degrees
- moved U7 43.4 mm to (192.3, 109.0), turned to 0 degrees
- moved R12 42.6 mm to (188.6, 111.2)
- moved IC1 42.3 mm to (184.0, 96.8), turned to 180 degrees
- moved CC_FLT1 42.0 mm to (184.9, 102.8), turned to 180 degrees
- moved R11 41.9 mm to (184.9, 104.4), turned to 180 degrees
- moved R10 41.8 mm to (184.9, 106.0), turned to 0 degrees
- moved U8 39.1 mm to (175.9, 97.4), turned to 180 degrees
- moved IC2 38.4 mm to (184.6, 108.8), turned to 0 degrees
- moved CC_Term1 36.6 mm to (179.9, 92.8), turned to 0 degrees
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Connections:
- C4 pad 1: +3.3V -> unconnected-(C4-Pad1)
- C4 pad 2: GND -> unconnected-(C4-Pad2)
- CC_Term1 pad 2: TelCAN_L -> TelCAN_L-
- CC_Term2 pad 2: CarCAN_L -> CarCAN_L-
- IC1 pad 6: TelCAN_L -> TelCAN_L-
- IC1 pad 7: TelCAN_H -> TelCAN_H+
- IC2 pad 6: CarCAN_L -> CarCAN_L-
- IC2 pad 7: CarCAN_H -> CarCAN_H+
- J4 pad 1: IMU_MOSI -> /Connector/TP1
- J4 pad 2: IMU_CS -> /Connector/TP4
- J4 pad 5: GPS_SCL -> GPS_SDA
- J4 pad 6: IMU_MISO -> /Connector/TP2
- J4 pad 7: GPS_SDA -> GPS_SCL
- J4 pad 8: IMU_CLK -> /Connector/TP5
- J5 pad 10: CarCAN_TX -> CarCAN_L-
- J5 pad 12: TelCAN_TX -> TelCAN_H+
- J5 pad 13: TelCAN_TX -> TelCAN_L-
- J5 pad 2: CarCAN_H -> CarCAN_H+
- J5 pad 3: CarCAN_RX -> CarCAN_L-
- J5 pad 5: TelCAN_RX -> TelCAN_H+
- J5 pad 6: TelCAN_RX -> TelCAN_L-
- J5 pad 9: CarCAN_TX -> CarCAN_H+
- J6 pad 1: IMU_INT1 -> IMU_CLK
- J6 pad 2: IMU_INT2 -> IMU_MOSI
- J6 pad 3: /Connector/TP1 -> IMU_CS
- J6 pad 4: /Connector/TP4 -> IMU_MISO
- J6 pad 5: /Connector/TP2 -> IMU_INT2
- J6 pad 6: /Connector/TP5 -> IMU_INT1
- J6 pad 7: /Connector/TP3 -> unconnected-(J6-Pin_7-Pad7)
- J6 pad 8: /Connector/TP6 -> unconnected-(J6-Pin_8-Pad8)
- J8 pad 11: CarCAN_RX -> TelCAN_TX
- J8 pad 5: CarCAN_TX -> TelCAN_RX
- J8 pad 7: TelCAN_TX -> CarCAN_RX
- J8 pad 9: TelCAN_RX -> CarCAN_TX
- J9 pad 10: /Connector/TP4 -> /Connector/TP2
- J9 pad 2: /Connector/TP2 -> /Connector/TP4
- R11 pad 1: unconnected-(R11-Pad1) -> /CAN/CarCAN_Fault
- R12 pad 2: CarCAN_H -> CarCAN_H+
- R22 pad 2: TelCAN_H -> TelCAN_H+
- U7 pad 1: CarCAN_H -> CarCAN_H+
- U7 pad 2: CarCAN_L -> CarCAN_L-
- U8 pad 1: TelCAN_H -> TelCAN_H+
- U8 pad 2: TelCAN_L -> TelCAN_L-
Routing:
- net TelCAN_L-: track 0.00 -> 74.1 mm
- net TelCAN_H+: track 0.00 -> 70.6 mm
- net CarCAN_H+: track 0.00 -> 50.6 mm
- net CarCAN_L-: track 0.00 -> 48.6 mm
- net IMU_INT2: track 0.00 -> 20.9 mm
- net IMU_INT1: track 0.00 -> 17.6 mm
- net IMU_CS: track 0.00 -> 14.8 mm
- net IMU_MISO: track 0.00 -> 12.9 mm
- net IMU_CLK: track 0.00 -> 7.10 mm
- net IMU_MOSI: track 0.00 -> 6.26 mm
- net +3V3: track 0.00 -> 5.08 mm
- net /GPS/+3.3V_GPS_BAT: track 0.00 -> 4.52 mm
- net /CAN/CarCAN_Fault: track 0.00 -> 3.43 mm
- net /CAN/TelCAN_Fault: track 0.00 -> 3.25 mm
- net /GPS/GPS_D8: track 0.00 -> 2.00 mm
- added copper zone on B.Cu, net GND
- added copper zone on F.Cu, net GND
Other:
- board outline added: 73.9 x 75.2 mm
- board text added: "21.59 mm (0.850 in)"
- board text added: "44.20 mm (1.748 in)"
- board text added: "67.41 mm (2.654 in)"
