File: TSOMProject.kicad_pcb (KiCad board)
At the start: 4 copper layers, 73.8 x 75.2 mm, 97 parts, among them IC1 TCAN337DCNR, IC2 TCAN337DCNR, IC3 LM74502HDDFR, J1 Conn_01x02, J10 Conn_02x04_Top_Bottom, J11 GPS_I2C, J13 Conn_02x03_Top_Bottom, J4 Conn_02x06_Counter_Clockwise, J6 To The Zedboard, J8 Conn_02x06_Odd_Even, Q5 NVMFWS1D7N04XMT1G, Q6 NVMFWS1D7N04XMT1G, SW4 GPS_RESET, U1 ASM330LHHTR, U2 CDSOT23-T24CAN, U3 LM61495RPHR, U7 CDSOT23-T24CAN, U9 PA1616S_GPS

Commit message: done antenna
Parts:
- added C31: 1u, Capacitor_SMD:C_0603_1608Metric_Pad1.08x0.95mm_HandSolder, F.Cu at (181.0, 108.3)
- added C32: 47p, Capacitor_SMD:C_0603_1608Metric_Pad1.08x0.95mm_HandSolder, F.Cu at (174.4, 106.8)
- added J2: RFPC-SMA28-F, TSOM Lib:GRADCONN_RFPC-SMA28-F, F.Cu at (177.8, 114.4)
- added J5: Conn_01x04, Connector_Molex:Molex_Nano-Fit_105310-xx04_2x02_P2.50mm_Vertical, F.Cu at (185.2, 146.4)
- added L2: 33n, Inductor_SMD:L_0603_1608Metric_Pad1.05x0.95mm_HandSolder, F.Cu at (177.7, 106.8)
- added R40: 10, Resistor_SMD:R_0603_1608Metric_Pad0.98x0.95mm_HandSolder, F.Cu at (181.0, 106.8)
- added TP10: TestPoint, TestPoint:TestPoint_THTPad_D2.0mm_Drill1.0mm, F.Cu at (205.6, 117.7)
- added TP11: TestPoint, TestPoint:TestPoint_THTPad_D2.0mm_Drill1.0mm, F.Cu at (205.6, 139.8)
- added TP12: TestPoint, TestPoint:TestPoint_THTPad_D2.0mm_Drill1.0mm, F.Cu at (205.6, 143.9)
- added TP5: TestPoint, TestPoint:TestPoint_THTPad_D2.0mm_Drill1.0mm, F.Cu at (205.6, 105.2)
- added TP6: TestPoint, TestPoint:TestPoint_THTPad_D2.0mm_Drill1.0mm, F.Cu at (205.6, 101.2)
- added TP7: TestPoint, TestPoint:TestPoint_THTPad_D2.0mm_Drill1.0mm, F.Cu at (205.6, 129.9)
- added TP8: TestPoint, TestPoint:TestPoint_THTPad_D2.0mm_Drill1.0mm, F.Cu at (205.6, 125.8)
- added TP9: TestPoint, TestPoint:TestPoint_THTPad_D2.0mm_Drill1.0mm, F.Cu at (205.6, 121.8)
- moved F1 10.0 mm to (184.5, 125.1)
- moved J1 0.06 mm to (185.2, 158.8)
Connections:
- J4 pad 1: /Connector/TP4 -> Net-(J4-Pin_1)
- J4 pad 2: /Connector/TP1 -> Net-(J4-Pin_2)
- J4 pad 3: unconnected-(J4-Pin_3-Pad3) -> Net-(J4-Pin_3)
- J4 pad 4: unconnected-(J4-Pin_4-Pad4) -> Net-(J4-Pin_4)
- J4 pad 6: /Connector/TP5 -> TelCAN_TX
- J4 pad 8: /Connector/TP2 -> TelCAN_RX
- J6 pad 7: unconnected-(J6-Pin_7-Pad7) -> Net-(J6-Pin_7)
- J6 pad 8: unconnected-(J6-Pin_8-Pad8) -> Net-(J6-Pin_8)
- J8 pad 11: unconnected-(J8-Pin_11-Pad11) -> Net-(J8-Pin_11)
- J8 pad 12: unconnected-(J8-Pin_12-Pad12) -> Net-(J8-Pin_12)
Routing:
- net TelCAN_TX: track 13.7 -> 37.9 mm
- net TelCAN_RX: track 6.41 -> 25.3 mm
- net +3V3: track 193.3 -> 210.8 mm, vias 0 -> 2
- net GND: track 14.8 -> 31.0 mm, vias 1040 -> 707
- net Net-(J4-Pin_2): track 0.00 -> 10.5 mm
- net Net-(J8-Pin_11): track 0.00 -> 9.83 mm
- net Net-(J4-Pin_4): track 0.00 -> 9.78 mm
- net Net-(J6-Pin_8): track 0.00 -> 9.75 mm
- net Net-(C32-Pad2): track 0.00 -> 9.66 mm
- net Net-(J4-Pin_1): track 0.00 -> 6.23 mm
- net Net-(J4-Pin_3): track 0.00 -> 5.64 mm
- net Net-(J8-Pin_12): track 0.00 -> 5.61 mm
- net Net-(J6-Pin_7): track 0.00 -> 5.53 mm
- net /GPS/GPS_EXT_OFF: track 0.00 -> 3.15 mm
- net Net-(C31-Pad1): track 0.00 -> 3.05 mm
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Other:
- board text added: "JE1"
- board text added: "JE7"
- board text removed: "${REFERENCE}"

Commit message: did some stuff
Parts:
- C31: value 1u -> 10n

Commit message: mika changes
Routing:
- net GND: track 31.0 -> 37.8 mm, vias 707 -> 708
- net +3V3: track 210.8 -> 214.7 mm
- net /GPS/GPS_D8: track 0.00 -> 1.54 mm
- net Net-(IC3-OV): track 8.07 -> 9.03 mm

Commit message: gerb
Parts:
- FB1: footprint Resistor_SMD:R_0402_1005Metric -> Inductor_SMD:L_0603_1608Metric_Pad1.05x0.95mm_HandSolder
- moved FB1 1.23 mm to (151.8, 92.9)
Routing:
- net +3V3: track 214.7 -> 211.1 mm
- net GPS_SCL: track 45.9 -> 46.7 mm
